Commit message: Add base_footprint link with a simple circle visualization for Rviz

File: turtlebot4_description/urdf/lite/turtlebot4.urdf.xacro (robot description, xacro)
@@ -27,3 +27,20 @@
     <origin xyz="${oakd_lite_x_offset} ${oakd_lite_y_offset} ${oakd_lite_z_offset}"/>
   </xacro:oakd>
+  <!-- Base footprint for navigation -->
+  <link name="base_footprint">
+    <visual>
+      <geometry>
+        <cylinder length="0.001" radius="${0.335/2}"/>
+      </geometry>
+      <material name="dark_grey">
+        <color rgba="0.1 0.1 0.1 1"/>
+      </material>
+    </visual>
+  </link>
+  <joint name="base_footprint_joint" type="fixed">
+    <!-- Create3's base_link is already on the ground -->
+    <origin xyz="0 0 0" rpy="0 0 0" />
+    <parent link="base_link" />
+    <child link="base_footprint" />
+  </joint>
 </robot>

File: turtlebot4_description/urdf/standard/turtlebot4.urdf.xacro (robot description, xacro)
@@ -101,3 +101,20 @@
     <origin xyz="${oakd_pro_x_offset} ${oakd_pro_y_offset} ${oakd_pro_z_offset}"/>
   </xacro:oakd>
+  <!-- Base footprint for navigation -->
+  <link name="base_footprint">
+    <visual>
+      <geometry>
+        <cylinder length="0.001" radius="${0.335/2}"/>
+      </geometry>
+      <material name="dark_grey">
+        <color rgba="0.1 0.1 0.1 1"/>
+      </material>
+    </visual>
+  </link>
+  <joint name="base_footprint_joint" type="fixed">
+    <!-- Create3's base_link is already on the ground -->
+    <origin xyz="0 0 0" rpy="0 0 0" />
+    <parent link="base_link" />
+    <child link="base_footprint" />
+  </joint>
 </robot>

Commit message: Remove the base_footprint visualization

File: turtlebot4_description/urdf/lite/turtlebot4.urdf.xacro (robot description, xacro)
@@ -28,14 +28,5 @@
   </xacro:oakd>
   <!-- Base footprint for navigation -->
-  <link name="base_footprint">
-    <visual>
-      <geometry>
-        <cylinder length="0.001" radius="${0.335/2}"/>
-      </geometry>
-      <material name="dark_grey">
-        <color rgba="0.1 0.1 0.1 1"/>
-      </material>
-    </visual>
-  </link>
+  <link name="base_footprint" />
   <joint name="base_footprint_joint" type="fixed">
     <!-- Create3's base_link is already on the ground -->

File: turtlebot4_description/urdf/standard/turtlebot4.urdf.xacro (robot description, xacro)
@@ -102,14 +102,5 @@
   </xacro:oakd>
   <!-- Base footprint for navigation -->
-  <link name="base_footprint">
-    <visual>
-      <geometry>
-        <cylinder length="0.001" radius="${0.335/2}"/>
-      </geometry>
-      <material name="dark_grey">
-        <color rgba="0.1 0.1 0.1 1"/>
-      </material>
-    </visual>
-  </link>
+  <link name="base_footprint" />
   <joint name="base_footprint_joint" type="fixed">
     <!-- Create3's base_link is already on the ground -->
